File: kicad/arcaduinome.sch (KiCad schematic (older format))
At the start: 0 parts

Commit message: added arduino and rgb led compenents; started placing components on schematic
Parts:
- added D? (x16): RGB_LED, symbol RGB_LED
- added Q? (x5): SLA5086, ~, symbol SLA5086
- added SW? (x16): SW_PUSH_SMALL, ~, symbol SW_PUSH_SMALL
- added U?: ARDUINO, symbol ARDUINO
- added U? (x2): STPIC6D595, ~, symbol STPIC6D595
